File: schematics/processorDesign/processorDesign.kicad_sch (KiCad schematic)
At the start: 73 parts

Commit message: added the IF stage and it's working properly
Connections:
- net CLK: now also U?. (instruction1), U?. (read_data), U?. (write_data), U?. (write_data)
- net EDU/mem_write_MEM: no longer U?. (write_data)
- net at U?. (select): no longer U?. (stall)
- net at U?. (select): now also U?. (stall) (x4)
- net at U?. (select): now also U?.2, U?.3, U?.3
- net at U?. (select): now also U?. (reset)
- net at U?. (select): now also U?.3
- new net: U?. (select), U?. (select), U?. (select), U?.3
- new net: U?. (out), U?. (stall) (x5)
- new net: U?. (select), U?. (stall) (x2)
- new net: U?. (stall), U?. (stall) (x12)
- new net: U?. (select), U?. (select)
- new net: U?. (read_data), U?. (stall)
- new net: U?. (stall), U?. (stall), U?.3
- new net: U?. (stall), U?. (write_data)
- new net: U?. (out), U?. (select) (x3)
- new net: U?. (reset), U?. (reset), U?. (select), U?.1
- new net: U?. (clk), U?. (select)
- new net: U?. (reset), U?. (stall)
- now unconnected: U?. (select)

Commit message: the ID stage and ID_EX buffer are now working correctly until further testing
Connections:
- net at U?. (select): no longer U?. (stall)
- net at U?. (select): now also U?. (stall) (x4)
- net at U?. (select): now also U?.2, U?.3, U?.3
- net at U?. (select): now also U?. (reset)
- net at U?. (select): now also U?.3
- new net: U?. (select), U?. (select), U?. (select), U?.3
- new net: U?. (out), U?. (stall) (x5)
- new net: U?. (select), U?. (stall) (x2)
- new net: U?. (stall), U?. (stall) (x12)
- new net: U?. (select), U?. (select)
- new net: U?. (read_data), U?. (stall)
- new net: U?. (stall), U?. (stall), U?.3
- new net: U?. (stall), U?. (write_data)
- new net: U?. (out), U?. (select) (x3)
- new net: U?. (reset), U?. (reset), U?. (select), U?.1
- new net: U?. (clk), U?. (select)
- new net: U?. (reset), U?. (stall)
- now unconnected: U?. (select)
Changed lines of the file:
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@@
   )
   (symbol (lib_id "computerArchProj:ID_EX") (at 838.2 356.87 0) (unit 1)
-    (in_bom yes) (on_board yes) (fields_autoplaced)
+    (in_bom yes) (on_board yes)
     (property "Reference" "U?" (id 0) (at 838.2 243.84 0)
       (effects (font (size 1.27 1.27)) hide)
     )
-    (property "Value" "ID_EX" (id 1) (at 838.2 246.38 0))
+    (property "Value" "ID_EX" (id 1) (at 838.2 252.73 0))
     (property "Footprint" "" (id 2) (at 838.2 270.51 0)
       (effects (font (size 1.27 1.27)) hide)
@@
   )
   (symbol (lib_id "computerArchProj:EX_MEM") (at 1532.89 384.81 0) (unit 1)
-    (in_bom yes) (on_board yes) (fields_autoplaced)
+    (in_bom yes) (on_board yes)
     (property "Reference" "U?" (id 0) (at 1532.89 327.66 0)
       (effects (font (size 1.27 1.27)) hide)
     )
-    (property "Value" "EX_MEM" (id 1) (at 1532.89 330.2 0))
+    (property "Value" "EX_MEM" (id 1) (at 1532.89 328.93 0))
     (property "Footprint" "" (id 2) (at 1532.89 347.98 0)
       (effects (font (size 1.27 1.27)) hide)

Commit message: the EX stage and EX_MEM is now complete till further testing
Parts:
- removed U? (x3): 4071, symbol 4xxx:4071
- added U? (x3): equality, symbol computerArchProj:equality
- added U?: 4073, symbol 4xxx:4073
- added U? (x3): 4075, symbol 4xxx:4075
- added U?: 4081, symbol 4xxx:4081
- added U?: 4071, symbol 4xxx:4071
Connections:
- net ALU/CF_in: now also U?.
- net ALU/CF_out: now also U?.
- net ALU/NF_in: now also U?.
- net ALU/NF_out: now also U?.
- net ALU/ZF_in: now also U?.
- net ALU/ZF_out: now also U?.
- net reset: now also U?.2, U?.2, U?.2, U?.2
- net at U?. (select): no longer U?. (stall)
- net at U?. (select): now also U?. (stall) (x4)
- net at U?. (select): now also U?.2, U?.3, U?.3
- net at U?. (select): now also U?. (reset)
- net at U?. (select): now also U?.3
- new net: U?.1, U?.3
- new net: U?. (out), U?. (stall) (x4)
- new net: U?. (stall), U?.1 (x4)
- new net: U?. (select), U?. (stall) (x2)
- new net: U?. (stall), U?. (stall) (x12)
- new net: U?. (select), U?. (select)
- new net: U?., U?.2
- new net: U?. (read_data), U?. (stall)
- new net: U?. (stall), U?. (stall), U?.3
- new net: U?., U?.8
- new net: U?. (stall), U?. (write_data)
- new net: U?. (out), U?. (select) (x3)
- new net: U?. (select), U?. (select), U?. (select), U?.3
- new net: U?., U?.1
- new net: U?.2, U?.9
- new net: U?. (out), U?.9 (x3)
- new net: U?. (out), U?.3
- new net: U?. (select), U?.8 (x3)
- new net: U?. (reset), U?. (reset), U?. (select), U?.1
- new net: U?. (clk), U?. (select)
- new net: U?. (reset), U?. (stall)
- now unconnected: U?. (select)
Other:
- note added: "flags + PC[28:0]"
- note removed: "flags + PC[29:0]"

Commit message: the MEM stage and MEM_WB buffer are now correctly working for command LDM and still under testing
Parts:
- removed U? (x3): 4081, symbol 4xxx:4081
- removed U?: 4071, symbol 4xxx:4071
- removed U? (x3): 74LS04, symbol 74xx:74LS04
- added U? (x4): 4081, symbol 4xxx:4081
- added U? (x2): 74LS04, symbol 74xx:74LS04
Connections:
- net CLK: no longer U?. (reset)
- net EDU/mem_read_MEM: now also U?.1
- net EDU/mem_write_MEM: now also U?. (write_data)
- net reset: now also U?. (reset)
- net at U?. (select): no longer U?. (stall)
- net at U?. (select): now also U?. (stall) (x4)
- net at U?. (select): now also U?.2, U?.3, U?.3
- net at U?. (select): now also U?. (reset)
- net at U?. (select): now also U?.3
- new net: U?. (reset), U?. (select), U?. (stall), U?. (stall), U?.2, U?.2, U?.3
- new net: U?. (stall), U?.1, U?.1, U?.2
- new net: U?.2, U?.2
- new net: U?. (reset), U?.3
- new net: U?. (out), U?. (stall) (x4)
- new net: U?. (select), U?. (stall) (x2)
- new net: U?. (stall), U?. (stall) (x12)
- new net: U?. (select), U?. (select)
- new net: U?. (read_data), U?. (stall)
- new net: U?. (stall), U?. (stall), U?.3
- new net: U?. (stall), U?. (write_data)
- new net: U?. (out), U?. (select) (x3)
- new net: U?. (select), U?. (select), U?. (select), U?.3
- new net: U?. (reset), U?.1, U?.1, U?.2
- new net: U?. (reset), U?. (reset), U?. (select), U?.1
- new net: U?. (clk), U?. (select)
- new net: U?.1, U?.2
- new net: U?. (reset), U?. (stall)
- new net: U?.2, U?.3
- now unconnected: U?. (select), U?. (select)
Other:
- note added: "PC[31:16] 16 bits width"
- note removed: "PC[32:16] 16 bits width"
