File: schematics/processorDesign/processorDesign.kicad_sch (KiCad schematic)
At the start: 79 parts

Commit message: edited the priority of the flags for the CCR
Parts:
- removed U? (x2): equality, symbol computerArchProj:equality
- removed U?: 4073, symbol 4xxx:4073
Connections:
- net ALU/NF_in: no longer U?.
- net ALU/NF_out: no longer U?.
- net CLK: no longer U?. (instruction1)
- net at U?. (select): no longer U?. (stall)
- net at U?. (select): now also U?. (stall) (x4)
- net at U?.: now also U?.2
- net at U?. (select): now also U?.2, U?.3, U?.3
- net at U?. (select): now also U?. (reset)
- net at U?. (select): now also U?.3
- new net: U?. (out), U?. (stall) (x4)
- new net: U?. (select), U?. (stall) (x2)
- new net: U?. (stall), U?. (stall) (x12)
- new net: U?. (select), U?. (select)
- new net: U?. (read_data), U?. (stall)
- new net: U?. (stall), U?. (stall), U?.3
- new net: U?. (stall), U?. (write_data)
- new net: U?. (out), U?. (select) (x3)
- new net: U?. (select), U?. (select), U?. (select), U?.3
- new net: U?. (reset), U?. (reset), U?. (select), U?.1
- new net: U?. (clk), U?. (select)
- new net: U?. (reset), U?. (stall)
- now unconnected: U?. (select)

Commit message: initially integrated processor without being tested
Parts:
- removed U?: 4075, symbol 4xxx:4075
- removed U?: 4072, symbol 4xxx:4072
- removed U?: 4071, symbol 4xxx:4071
- added U?: mux_4x2, symbol computerArchProj:mux_4x2
- added U?: CAUSE, symbol computerArchProj:reg
- added U? (x4): 4071, symbol 4xxx:4071
- added U?: 4075, symbol 4xxx:4075
- added U?: reset, symbol computerArchProj:register
- added U?: INT, symbol computerArchProj:register
Connections:
- net CLK: now also U?. (out), U?. (out)
- net EDU/exception: now also U?. (reset), U?.2
- net EDU/is_jmp_EX: no longer U?. (select), U?. (select), U?. (select), U?.1
- net EDU/mem_read_MEM: no longer U?. (stall), U?. (write_data), U?.1
- net EDU/mem_write_MEM: no longer U?. (stall), U?. (write_data)
- net HDU/stall: now also U?.8
- net interrupt: now also U?. (out); no longer U?. (stall), U?.2
- net reset: now also U?. (reset), U?. (stall), U?. (stall), U?. (out), U?. (reset); no longer U?.1
- net at U?.1: now also U?.3; no longer U?. (stall)
- net at U?.1, U?.1, U?.2: now also U?.3; no longer U?. (stall)
- net at U?. (select): no longer U?. (stall)
- net at U?. (select): now also U?. (stall), U?.1, U?.1
- net at U?.: now also U?.2
- net at U?.3: now also U?.1
- net at U?. (select): now also U?.2, U?.3, U?.2
- net at U?. (select): now also U?. (reset)
- net at U?. (select): now also U?. (stall) (x3)
- net at U?. (select): now also U?.3
- net at U?. (select): now also U?.8
- new net: U?. (reset), U?. (reset), U?. (select), U?. (stall), U?. (stall), U?.2, U?.2, U?.3
- new net: U?. (out), U?. (stall) (x4)
- new net: U?. (select), U?. (stall) (x2)
- new net: U?. (stall), U?. (stall) (x12)
- new net: U?. (stall), U?.9
- new net: U?. (select), U?. (select)
- new net: U?. (read_data), U?. (stall)
- new net: U?. (stall), U?. (stall), U?.3
- new net: U?. (out), U?. (stall), U?.2
- new net: U?. (stall), U?.3
- new net: U?. (stall), U?. (write_data) (x2)
- new net: U?. (out), U?. (select) (x3)
- new net: U?. (select), U?. (select), U?. (select), U?.3
- new net: U?. (select), U?. (select), U?. (select), U?.1
- new net: U?. (reset), U?. (reset), U?. (select), U?.1
- new net: U?. (clk), U?. (select)
- new net: U?. (stall), U?.2 (x2)
- new net: U?. (stall), U?. (write_data), U?.1
- new net: U?. (reset), U?. (stall)
- new net: U?.1, U?.3
- new net: U?. (out), U?.1
- new net CAUSE: U?. (reset)
- new net EDU/exception_EXE: U?.2
- new net EDU/exception_MEM: U?. (stall), U?.1
- now unconnected: U?. (select), U?. (select)
- no-connect marks 5 -> 6
Other:
- sheet EDU ports: added CAUSE, PC_src, exception_EXE, exception_ID, exception_MEM, instr_opcode; removed none
- note added: "instr[15:12] 4 bits width (opcode)"
- title: (none) -> RAYZEN 15

Commit message: test12
Parts:
- removed U? (x2): 4071, symbol 4xxx:4071
- added U?: 4071, symbol 4xxx:4071
Connections:
- net CU/CLR_INT is gone; now on net reset: U?. (stall)
- net CU/SET_INT: now also U?.1; no longer U?. (stall)
- net interrupt: now also U?.2; no longer U?. (out)
- net at U?. (select): no longer U?. (stall)
- net at U?. (select): now also U?. (stall), U?.1, U?.1
- net at U?.: now also U?.2
- net at U?. (select): now also U?.2, U?.2, U?.3
- net at U?. (select): now also U?. (reset)
- net at U?. (select): now also U?. (stall) (x3)
- net at U?. (select): now also U?.3
- net at U?. (select): now also U?.8
- new net: U?. (reset), U?. (reset), U?. (select), U?. (stall), U?. (stall), U?.2, U?.2, U?.3
- new net: U?. (stall), U?. (stall) (x13)
- new net: U?. (out), U?. (stall) (x4)
- new net: U?. (select), U?. (stall) (x2)
- new net: U?. (select), U?. (select)
- new net: U?. (read_data), U?. (stall)
- new net: U?. (stall), U?. (stall), U?.3
- new net: U?. (out), U?. (select), U?. (stall)
- new net: U?. (stall), U?. (write_data) (x2)
- new net: U?. (out), U?. (select) (x3)
- new net: U?. (select), U?. (select), U?. (select), U?.3
- new net: U?. (select), U?. (select), U?. (select), U?.1
- new net: U?. (reset), U?. (reset), U?. (select), U?.1
- new net: U?. (clk), U?. (select)
- new net: U?. (stall), U?. (write_data), U?.1
- new net: U?. (reset), U?. (stall)
- new net: U?. (out), U?.3
- new net CU/CLR_OVF: U?. (stall)
- new net CU/SET_OVF: U?. (stall)
- now unconnected: U?. (select), U?. (select), U?. (select)
Other:
- sheet CU ports: added CLR_OVF, SET_OVF; removed CLR_INT

Commit message: the interrupt is now working correctly
Parts:
- removed U? (x2): 4081, symbol 4xxx:4081
- added U? (x4): 4071, symbol 4xxx:4071
- added U? (x2): mux_2x1, symbol computerArchProj:mux_2x1
- added U?: 4081, symbol 4xxx:4081
- added U?: 74LS04, symbol 74xx:74LS04
- added U? (x2): 4073, symbol 4xxx:4073
- added U?: 4075, symbol 4xxx:4075
- added U?: Sub, symbol computerArchProj:Sub
Connections:
- net CU/memWrite: now also U?.1; no longer U?. (stall)
- net CU/mem_address_src: now also U?.1; no longer U?. (stall)
- net CU/mem_data_src: now also U?.1; no longer U?. (stall)
- net reset: now also U?.8; no longer U?. (reset), U?. (reset)
- net at U?.3: now also U?.1
- net at U?.1: now also U?.9
- net at U?. (select): no longer U?. (stall)
- net at U?. (select): now also U?. (stall), U?.1, U?.1, U?. (select)
- net at U?.: now also U?.2
- net at U?. (select): now also U?.2, U?.2, U?.3
- net at U?.2: now also U?.1, U?.1
- net at U?. (select): now also U?. (reset)
- net at U?. (select): now also U?. (stall) (x3)
- net at U?.1, U?.3: now also U?.1
- net at U?. (select): now also U?.3
- net at U?. (select): now also U?.8
- new net: U?. (stall), U?. (stall), U?.2, U?.2, U?.2
- new net: U?. (stall), U?.3 (x4)
- new net: U?. (reset), U?. (reset), U?. (select), U?. (stall), U?. (stall), U?.2, U?.3, U?.8
- new net: U?. (out), U?. (stall) (x4)
- new net: U?. (select), U?. (stall) (x2)
- new net: U?. (stall), U?. (stall) (x12)
- new net: U?. (select), U?. (select)
- new net: U?. (select), U?. (select), U?. (select), U?. (select), U?.3
- new net: U?. (out), U?. (select) (x4)
- new net: U?. (read_data), U?. (stall)
- new net: U?. (stall), U?. (stall), U?. (stall), U?.2, U?.3
- new net: U?. (select), U?. (stall), U?. (stall), U?.1, U?.2, U?.2
- new net: U?. (stall), U?. (write_data) (x2)
- new net: U?. (select), U?. (select), U?. (select), U?.1
- new net: U?. (reset), U?. (reset), U?.1, U?.1
- new net: U?. (clk), U?. (select)
- new net: U?. (select), U?.3
- new net: U?.2, U?.2
- new net: U?. (reset), U?. (reset), U?.9
- new net: U?. (stall), U?. (write_data), U?.1, U?.2
- new net: U?. (reset), U?. (stall)
- new net ALU/OVF_in: U?. (out)
- new net ALU/OVF_out: U?. (select)
- now unconnected: U?. (select), U?. (select), U?. (select), U?. (select)
Other:
- sheet ALU ports: added OVF_in, OVF_out; removed none
- note added: "1 bit width (OVF)"
- note added: "28 bit width"
- note added: "4 bit width (flags)"
- note added: "4 bits width (flags)"
- note added: "PC[27:0] 28 bits width"
- note added: "PC[31:28] 4 bits width (flags)"
- note added: "flags + PC[27:0]"
- note removed: "3 bit width (flags)"
- note removed: "3 bits width (flags)"
- note removed: "flags + PC[28:0]"

Commit message: the processor is up and running tested and verified, need only tests for some bonus instructions like all I_types instruction except LDM , MUL , DIV , testing EDU and HDU
Parts:
- removed U? (x2): mux_2x1, symbol computerArchProj:mux_2x1
- removed U? (x5): 4075, symbol 4xxx:4075
- removed U?: sign_extend, symbol computerArchProj:sign_extend
- removed U? (x2): 4071, symbol 4xxx:4071
- added U? (x6): mux_2x1, symbol computerArchProj:mux_2x1
- added U? (x2): 4072, symbol 4xxx:4072
- added U? (x3): 4071, symbol 4xxx:4071
- added U?: JMP, symbol computerArchProj:register
- added U? (x3): 4075, symbol 4xxx:4075
- added U?: sign_extend, symbol computerArchProj:sign_extend
Connections:
- net CLK: now also U?. (stall)
- net EDU/exception: now also U?.8
- net EDU/exception_MEM: now also U?.8; no longer U?. (stall)
- net HDU/stall: now also U?.4
- net reset: now also U?.2, U?.2, U?.2, U?.2, U?.2, U?.5, U?.5; no longer U?. (stall), U?. (stall), U?. (stall)
- net GND: now reaches U?. (out), U?. (stall)
- net GND: now also U?. (stall), U?. (stall), U?. (stall)
- net at U?. (select): no longer U?. (stall)
- net at U?. (select): now also U?. (select), U?. (stall), U?.1, U?.1
- net at U?.: now also U?.2
- net at U?. (select), U?.2, U?.3: now also U?.1, U?.3
- net at U?. (select): now also U?. (reset) (x2)
- net at U?. (select): now also U?. (stall) (x3)
- net at U?.3: now also U?.1, U?.2
- net at U?. (select): now also U?.3
- net at U?.3: now also U?.2
- removed net forward_unit2/mem_to_Reg_WB: U?. (reset), U?. (select)
- new net: U?. (stall), U?.1 (x4)
- new net: U?. (reset), U?. (reset), U?. (select), U?. (stall), U?. (stall), U?.2, U?.3, U?.8
- new net: U?. (out), U?. (stall) (x4)
- new net: U?. (select), U?. (stall) (x2)
- new net: U?. (stall), U?. (stall) (x12)
- new net: U?. (select), U?. (select)
- new net: U?. (select), U?. (select), U?. (select), U?. (select), U?.3
- new net: U?. (out), U?. (select) (x7)
- new net: U?. (read_data), U?. (stall)
- new net: U?. (out), U?.3 (x3)
- new net: U?. (select), U?. (stall), U?. (stall), U?.1, U?.4, U?.8
- new net: U?. (stall), U?. (stall), U?. (stall), U?.2, U?.3
- new net: U?. (stall), U?.9 (x2)
- new net: U?. (select), U?. (stall), U?.1, U?.2, U?.3
- new net: U?. (select), U?. (select), U?. (stall)
- new net: U?. (reset), U?. (reset), U?.1, U?.1
- new net: U?. (select), U?.9
- new net: U?. (stall), U?. (write_data) (x2)
- new net: U?. (reset), U?. (reset), U?.1
- new net: U?. (clk), U?. (select)
- new net: U?. (reset), U?. (stall)
- new net forward_unit2/forward_Rdst1_to_address: U?. (select)
- new net forward_unit2/forward_Rdst1_to_write_data: U?. (select), U?. (select)
- new net forward_unit2/forward_Rdst2_to_address: U?. (select)
- new net forward_unit2/forward_Rdst2_to_write_data: U?. (select), U?. (select)
- now unconnected: U?. (select), U?. (select), U?. (select), U?. (select), U?. (select), U?. (select), U?. (select)
Other:
- sheet forward_unit2 ports: added forward_Rdst1_to_address, forward_Rdst1_to_write_data, forward_Rdst2_to_address, forward_Rdst2_to_write_data, reg_high_write_WB, reg_low_write_WB; removed forward_data_to_address, forward_data_to_write_data, mem_to_Reg_WB

Commit message: the processor is now up and running , tested and verified , except for the part related to labels due to a bug in the assembler
Parts:
- removed U?: 4072, symbol 4xxx:4072
- added U?: 4075, symbol 4xxx:4075
Connections:
- net GND: no longer U?. (stall)
- net HDU/stall: now also U?. (stall)
- net reset: now also U?.8
- net at U?. (select): no longer U?. (stall)
- net at U?. (select): now also U?. (select), U?. (stall), U?.1, U?.1
- net at U?.: now also U?.2
- net at U?.3: now also U?.1
- net at U?. (select), U?.1, U?.2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: now also U?.2
- net at U?. (select): no longer U?. (out)
- net at U?. (select): now also U?. (reset) (x2)
- net at U?. (select): now also U?. (stall) (x3)
- net at U?. (select): now also U?.3
- new net: U?. (reset), U?. (reset), U?. (select), U?. (stall), U?. (stall), U?.2, U?.3, U?.8
- new net: U?. (out), U?. (stall) (x4)
- new net: U?. (select), U?. (stall) (x2)
- new net: U?. (stall), U?.9
- new net: U?. (stall), U?. (stall) (x12)
- new net: U?. (select), U?. (select)
- new net: U?. (select), U?. (select), U?. (select), U?. (select), U?.3
- new net: U?. (out), U?. (select) (x7)
- new net: U?. (read_data), U?. (stall)
- new net: U?. (stall), U?. (stall), U?. (stall), U?.2, U?.3
- new net: U?. (select), U?. (select), U?. (stall)
- new net: U?. (stall), U?. (write_data) (x2)
- new net: U?. (reset), U?. (reset), U?.1
- new net: U?. (clk), U?. (select)
- new net: U?. (reset), U?. (stall)
- now unconnected: U?. (select), U?. (select), U?. (select), U?. (select), U?. (select)

Commit message: the processor is now up and running , tested and verified completly for almost most of the things
Parts:
- removed U? (x4): 4071, symbol 4xxx:4071
- added U? (x2): 4071, symbol 4xxx:4071
- added U? (x3): Sub, symbol computerArchProj:Sub
- added U?: 4081, symbol 4xxx:4081
Connections:
- net reset: now also U?.1; no longer U?. (reset), U?. (reset), U?. (reset), U?. (reset), U?. (reset), U?. (reset), U?. (select), U?. (stall), U?. (write_data), U?. (write_data), U?.2, U?.2, U?.5, U?.8
- net at U?.1, U?.1, U?.2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: now also U?.1
- net register file/reset: now reaches U?. (stall)
- net register file/reset: now also U?. (reset), U?. (reset), U?. (reset), U?. (reset), U?. (reset), U?. (reset), U?. (select), U?. (stall), U?. (write_data), U?. (write_data), U?.2, U?.2, U?.5, U?.8, U?.3; no longer U?. (stall)
- net at U?. (select): no longer U?. (stall)
- net at U?. (select): now also U?. (select), U?. (stall), U?.1, U?.1
- net at U?.: now also U?.2
- net at U?. (select): now also U?.1, U?.2, U?.2, U?.3
- net at U?. (select): no longer U?. (out)
- net at U?. (select): now also U?. (reset) (x2)
- net at U?.1, U?.3: now also U?.2
- net at U?. (select): now also U?. (stall) (x3)
- net at U?. (select): now also U?.3
- net at U?. (stall), U?. (write_data), U?.1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: now also U?.1
- new net: U?. (reset), U?. (reset), U?. (select), U?. (stall), U?. (stall), U?.2, U?.3, U?.8
- new net: U?. (stall), U?. (stall) (x20)
- new net: U?. (select), U?. (stall) (x9)
- new net: U?. (select), U?. (select)
- new net: U?. (select), U?. (select), U?. (select), U?. (select), U?.3
- new net: U?. (read_data), U?. (stall)
- new net: U?. (stall), U?. (stall), U?. (stall), U?.2, U?.3
- new net: U?. (select), U?. (select), U?. (stall)
- new net: U?. (stall), U?. (write_data) (x2)
- new net: U?. (reset), U?. (reset), U?.1
- new net: U?. (stall), U?.3
- new net: U?.2, U?.3
- new net: U?. (clk), U?. (select)
- new net: U?. (reset), U?. (stall)
- new net CU/RST: U?.2
- now unconnected: U?. (select), U?. (select), U?. (select), U?. (select), U?. (select)
Other:
- sheet CU ports: added RST; removed none

Commit message: added small code to EDU
Connections:
- net at U?. (select): no longer U?. (stall) (x2)
- net at U?. (select): now also U?. (select), U?. (stall), U?.1, U?.1
- net at U?.: now also U?.2
- net at U?. (select): now also U?.1, U?.2, U?.2, U?.3
- net at U?. (select): now also U?. (reset) (x2)
- net at U?. (select): now also U?. (stall) (x3)
- net at U?. (select): now also U?.3
- new net: U?. (reset), U?. (reset), U?. (select), U?. (stall), U?. (stall), U?.2, U?.3, U?.8
- new net: U?. (stall), U?. (stall) (x20)
- new net: U?. (select), U?. (stall) (x9)
- new net: U?. (select), U?. (select)
- new net: U?. (select), U?. (select), U?. (select), U?. (select), U?.3
- new net: U?. (read_data), U?. (stall)
- new net: U?. (stall), U?. (stall), U?. (stall), U?.2, U?.3
- new net: U?. (select), U?. (select), U?. (stall)
- new net: U?. (stall), U?. (write_data) (x2)
- new net: U?. (reset), U?. (reset), U?.1
- new net: U?. (clk), U?. (select)
- new net: U?. (reset), U?. (stall)
- now unconnected: U?. (select), U?. (select), U?. (select), U?. (select), U?. (select)
Changed lines of the file:
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@@
       (reference "U?") (unit 1) (value "4081") (footprint "")
+    )
+    (path "/24beea0c-0a1d-42e3-a6b3-fb99efb07535/07cd708a-7162-4979-9d04-8d76b2d1d604"
+      (reference "U?") (unit 1) (value "4071") (footprint "")
     )
     (path "/c77b66d9-6f44-4dfc-987d-6b034fc7555a/08bb51a3-92ff-43b2-9a87-e0e034672b60"
@@
       (reference "U?") (unit 1) (value "mux_4x2") (footprint "")
     )
+    (path "/24beea0c-0a1d-42e3-a6b3-fb99efb07535/173ece8b-ed4f-4e84-925b-396eea7eceaa"
+      (reference "U?") (unit 1) (value "equality") (footprint "")
+    )
     (path "/17d5ac74-1abe-483b-a4b4-7841ce28761a"
