File: schematics/processorDesign/processorDesign.kicad_sch (KiCad schematic)
At the start: 99 parts

Commit message: solved the problem of flush due to exception
Parts:
- removed U? (x3): 4075, symbol 4xxx:4075
- removed U?: 4071, symbol 4xxx:4071
- added U? (x5): 4071, symbol 4xxx:4071
Connections:
- net EDU/exception: now also U?. (stall), U?.1
- net EDU/exception_MEM: now also U?. (stall)
- net GND: no longer U?. (stall), U?. (stall)
- net HDU/stall: now also U?.2; no longer U?. (stall)
- net register file/reset: now also U?.2, U?.2, U?.2; no longer U?. (reset), U?. (stall), U?.5
- net at U?. (select): no longer U?. (stall) (x2)
- net at U?. (select): now also U?. (select), U?. (stall), U?.1, U?.1
- net at U?.: now also U?.2
- net at U?. (select), U?.2, U?.3: now also U?.1, U?.1
- net at U?.2, U?.3: now also U?.1
- net at U?. (select): now also U?. (reset) (x2)
- net at U?.3: now also U?.1
- net at U?. (select): now also U?. (stall) (x4)
- new net: U?. (stall), U?.3 (x4)
- new net: U?. (reset), U?. (reset), U?. (select), U?. (stall), U?. (stall), U?.2, U?.3, U?.8
- new net: U?. (stall), U?. (stall) (x20)
- new net: U?. (select), U?. (stall) (x9)
- new net: U?. (select), U?. (select)
- new net: U?. (select), U?. (select), U?. (select), U?. (select), U?.3
- new net: U?. (read_data), U?. (stall)
- new net: U?. (stall), U?. (stall), U?. (stall), U?.2, U?.3
- new net: U?. (select), U?. (select), U?. (stall)
- new net: U?. (stall), U?. (write_data) (x2)
- new net: U?. (reset), U?. (stall), U?.2, U?.3, U?.5
- new net: U?. (reset), U?. (reset), U?.1
- new net: U?. (clk), U?. (select)
- new net: U?. (reset), U?. (stall)
- now unconnected: U?. (select), U?. (select), U?. (select), U?. (select), U?. (select)
