File: schematics/processorDesign/ALU.kicad_sch (KiCad schematic)
At the start: 17 parts

Commit message: added the IF stage and it's working properly
Connections:
- net at U?. (Z): now also U?. (select) (x6)
- net at U. (Z): now also U?. (select); no longer U?. (select) (x2)
- net at U?. (Z): now also U?. (select); no longer U?. (select) (x2)
- new net: U?. (Z), U?. (select) (x11)
- new net: U?. (Z), U?. (select), U?. (select)
- new net: U. (Z), U?. (select) (x4)
- now unconnected: U?. (select)

Commit message: the ID stage and ID_EX buffer are now working correctly until further testing
Connections:
- net at U?. (Z): now also U?. (select) (x6)
- net at U. (Z): now also U?. (select); no longer U?. (select) (x2)
- net at U?. (Z): now also U?. (select); no longer U?. (select) (x2)
- new net: U?. (Z), U?. (select) (x11)
- new net: U?. (Z), U?. (select), U?. (select)
- new net: U. (Z), U?. (select) (x4)
- now unconnected: U?. (select)

Commit message: the EX stage and EX_MEM is now complete till further testing
Connections:
- net at U?. (Z): now also U?. (select) (x6)
- net at U. (Z): now also U?. (select); no longer U?. (select) (x2)
- net at U?. (Z): now also U?. (select); no longer U?. (select) (x2)
- new net: U?. (Z), U?. (select) (x11)
- new net: U?. (Z), U?. (select), U?. (select)
- new net: U. (Z), U?. (select) (x4)
- now unconnected: U?. (select)

Commit message: the MEM stage and MEM_WB buffer are now correctly working for command LDM and still under testing
Connections:
- net at U?. (Z): now also U?. (select) (x6)
- net at U. (Z): now also U?. (select); no longer U?. (select) (x2)
- net at U?. (Z): now also U?. (select); no longer U?. (select) (x2)
- new net: U?. (Z), U?. (select) (x11)
- new net: U?. (Z), U?. (select), U?. (select)
- new net: U. (Z), U?. (select) (x4)
- now unconnected: U?. (select)

Commit message: the pipeline processor is semi-working for phase 1 to be complete, just there is a small bug in the command called std
Connections:
- net at U?. (Z): now also U?. (select) (x6)
- net at U. (Z): now also U?. (select); no longer U?. (select) (x2)
- net at U?. (Z): now also U?. (select); no longer U?. (select) (x2)
- new net: U?. (Z), U?. (select) (x11)
- new net: U?. (Z), U?. (select), U?. (select)
- new net: U. (Z), U?. (select) (x4)
- now unconnected: U?. (select)

Commit message: edited the priority of the flags for the CCR
Connections:
- net at U?. (Z): now also U?. (select) (x6)
- net at U. (Z): now also U?. (select); no longer U?. (select) (x2)
- net at U?. (Z): now also U?. (select); no longer U?. (select) (x2)
- new net: U?. (Z), U?. (select) (x11)
- new net: U?. (Z), U?. (select), U?. (select)
- new net: U. (Z), U?. (select) (x4)
- now unconnected: U?. (select)

Commit message: initially integrated processor without being tested
Connections:
- net at U?. (Z): now also U?. (select) (x6)
- net at U. (Z): now also U?. (select); no longer U?. (select) (x2)
- net at U?. (Z): now also U?. (select); no longer U?. (select) (x2)
- new net: U?. (Z), U?. (select) (x11)
- new net: U?. (Z), U?. (select), U?. (select)
- new net: U. (Z), U?. (select) (x4)
- now unconnected: U?. (select)

Commit message: test12
Connections:
- net at U?. (Z): now also U?. (select) (x6)
- net at U. (Z): now also U?. (select); no longer U?. (select) (x2)
- net at U?. (Z): now also U?. (select); no longer U?. (select) (x2)
- new net: U?. (Z), U?. (select) (x11)
- new net: U?. (Z), U?. (select), U?. (select)
- new net: U. (Z), U?. (select) (x4)
- now unconnected: U?. (select)
