File: schematics/processorDesign/HazardDetectionUnit.kicad_sch (KiCad schematic)
At the start: 9 parts

Commit message: added the IF stage and it's working properly
Connections:
- net at U?.: now also U?.4
- net at U?.: now also U?.3
- net at U?.: now also U?.1
- net at U?.: now also U?.2

Commit message: the ID stage and ID_EX buffer are now working correctly until further testing
Connections:
- net at U?.: now also U?.4
- net at U?.: now also U?.3
- net at U?.: now also U?.1
- net at U?.: now also U?.2

Commit message: the EX stage and EX_MEM is now complete till further testing
Connections:
- net at U?.: now also U?.4
- net at U?.: now also U?.3
- net at U?.: now also U?.1
- net at U?.: now also U?.2

Commit message: the MEM stage and MEM_WB buffer are now correctly working for command LDM and still under testing
Connections:
- net at U?.: now also U?.4
- net at U?.: now also U?.3
- net at U?.: now also U?.1
- net at U?.: now also U?.2

Commit message: the pipeline processor is semi-working for phase 1 to be complete, just there is a small bug in the command called std
Connections:
- net at U?.: now also U?.4
- net at U?.: now also U?.3
- net at U?.: now also U?.1
- net at U?.: now also U?.2

Commit message: edited the priority of the flags for the CCR
Connections:
- net at U?.: now also U?.4
- net at U?.: now also U?.3
- net at U?.: now also U?.1
- net at U?.: now also U?.2

Commit message: initially integrated processor without being tested
Connections:
- net at U?.: now also U?.4
- net at U?.: now also U?.3
- net at U?.: now also U?.1
- net at U?.: now also U?.2

Commit message: test12
Connections:
- net at U?.: now also U?.4
- net at U?.: now also U?.3
- net at U?.: now also U?.1
- net at U?.: now also U?.2
