File: schematics/processorDesign/execprtionUnit.kicad_sch (KiCad schematic)
At the start: 12 parts

Commit message: added the IF stage and it's working properly
Connections:
- net at U?.: now also U?.1

Commit message: the ID stage and ID_EX buffer are now working correctly until further testing
Connections:
- net at U?.: now also U?.1

Commit message: the EX stage and EX_MEM is now complete till further testing
Connections:
- net at U?.: now also U?.1

Commit message: the MEM stage and MEM_WB buffer are now correctly working for command LDM and still under testing
Connections:
- net at U?.: now also U?.1

Commit message: the pipeline processor is semi-working for phase 1 to be complete, just there is a small bug in the command called std
Connections:
- net at U?.: now also U?.1

Commit message: edited the priority of the flags for the CCR
Connections:
- net at U?.: now also U?.1

Commit message: initially integrated processor without being tested
Parts:
- added U? (x3): 4071, symbol 4xxx:4071
- added U? (x9): mux_2x1, symbol computerArchProj:mux_2x1
- added U?: cmp, symbol computerArchProj:cmp
Connections:
- net exception: now also U?.3; no longer U?.1
- net at U?.3, U?.4: now also U?. (select), U?.2
- net at U?.: now also U?.1
- net at U?.2, U?.3: now also U?. (select), U?.1
- net at U?.3, U?.3: now also U?.1
- net at U?.3, U?.5: now also U?. (select), U?.2
- net at U?., U?.1: now also U?. (select)
- net at U?., U?.2: now also U?. (select)
- new net: U?.1, U?.1
- new net exception_EXE: U?. (select), U?.3
- new net exception_ID: U?., U?. (select), U?. (select), U?.2
- new net exception_MEM: U?. (select), U?.3
Other:
- note added: "2 bits width"
- note added: "3 bits width"

Commit message: test12
Connections:
- net at U?.: now also U?.1
- new net: U?., U?. (select), U?.1
- new net: U?., U?. (select), U?.2
- now unconnected: U?., U?., U?. (select), U?. (select)
