File: schematics/processorDesign/forward_unit1.kicad_sch (KiCad schematic)
At the start: 24 parts

Commit message: the interrupt is now working correctly
Connections:
- net at U?.: now also U?.1 (x5)
- net at U?. (select): now also U?.3

Commit message: the processor is now up and running , tested and verified , except for the part related to labels due to a bug in the assembler
Connections:
- net at U?.: now also U?.1 (x5)
- net at U?. (select): now also U?.3

Commit message: the processor is now up and running , tested and verified completly for almost most of the things
Connections:
- net at U?.: now also U?.1 (x5)
- net at U?. (select): now also U?.3

Commit message: added small code to EDU
Connections:
- net at U?.: now also U?.1 (x5)
- net at U?. (select): now also U?.3
