File: schematics/processorDesign/regFile.kicad_sch (KiCad schematic)
At the start: 31 parts

Commit message: added the IF stage and it's working properly
Connections:
- net at U?. (select): now also U?. (in), U?. (select) (x3)
- net at U?. (select): now also U?. (in), U?. (select); no longer U. (reset) (x2)
- net at U?. (select): now also U. (reset); no longer U?. (in) (x5)
- net at U?. (in): now also U?. (select); no longer U?. (select)
- net at U?. (in): now also U?.3
- net at U?. (select): now also U?. (in), U?. (select); no longer U?. (in)
- new net: U. (reset), U?. (select) (x3)
- new net: U?. (in), U?. (select) (x15)
- new net: U?. (in), U?. (select), U?. (select) (x2)
- now unconnected: U?. (select), U?. (select), U?. (select), U?. (select), U?. (select)

Commit message: the ID stage and ID_EX buffer are now working correctly until further testing
Connections:
- net at U?. (select): now also U?. (in), U?. (select) (x3)
- net at U?. (select): now also U?. (in), U?. (select); no longer U. (reset) (x2)
- net at U?. (select): now also U. (reset); no longer U?. (in) (x5)
- net at U?. (in): now also U?. (select); no longer U?. (select)
- net at U?. (in): now also U?.3
- net at U?. (select): now also U?. (in), U?. (select); no longer U?. (in)
- new net: U. (reset), U?. (select) (x3)
- new net: U?. (in), U?. (select) (x15)
- new net: U?. (in), U?. (select), U?. (select) (x2)
- now unconnected: U?. (select), U?. (select), U?. (select), U?. (select), U?. (select)

Commit message: the EX stage and EX_MEM is now complete till further testing
Connections:
- net at U?. (select): now also U?. (in), U?. (select) (x3)
- net at U?. (select): now also U?. (in), U?. (select); no longer U. (reset) (x2)
- net at U?. (select): now also U. (reset); no longer U?. (in) (x5)
- net at U?. (in): now also U?. (select); no longer U?. (select)
- net at U?. (in): now also U?.3
- net at U?. (select): now also U?. (in), U?. (select); no longer U?. (in)
- new net: U. (reset), U?. (select) (x3)
- new net: U?. (in), U?. (select) (x15)
- new net: U?. (in), U?. (select), U?. (select) (x2)
- now unconnected: U?. (select), U?. (select), U?. (select), U?. (select), U?. (select)

Commit message: the MEM stage and MEM_WB buffer are now correctly working for command LDM and still under testing
Connections:
- net at U?. (select): now also U?. (in), U?. (select) (x3)
- net at U?. (select): now also U?. (in), U?. (select); no longer U. (reset) (x2)
- net at U?. (select): now also U. (reset); no longer U?. (in) (x5)
- net at U?. (in): now also U?. (select); no longer U?. (select)
- net at U?. (in): now also U?.3
- net at U?. (select): now also U?. (in), U?. (select); no longer U?. (in)
- new net: U. (reset), U?. (select) (x3)
- new net: U?. (in), U?. (select) (x15)
- new net: U?. (in), U?. (select), U?. (select) (x2)
- now unconnected: U?. (select), U?. (select), U?. (select), U?. (select), U?. (select)

Commit message: the pipeline processor is semi-working for phase 1 to be complete, just there is a small bug in the command called std
Connections:
- net at U?. (select): now also U?. (in), U?. (select) (x3)
- net at U?. (select): now also U?. (in), U?. (select); no longer U. (reset) (x2)
- net at U?. (select): now also U. (reset); no longer U?. (in) (x5)
- net at U?. (in): now also U?. (select); no longer U?. (select)
- net at U?. (in): now also U?.3
- net at U?. (select): now also U?. (in), U?. (select); no longer U?. (in)
- new net: U. (reset), U?. (select) (x3)
- new net: U?. (in), U?. (select) (x15)
- new net: U?. (in), U?. (select), U?. (select) (x2)
- now unconnected: U?. (select), U?. (select), U?. (select), U?. (select), U?. (select)

Commit message: edited the priority of the flags for the CCR
Connections:
- net at U?. (select): now also U?. (in), U?. (select) (x3)
- net at U?. (select): now also U?. (in), U?. (select); no longer U. (reset) (x2)
- net at U?. (select): now also U. (reset); no longer U?. (in) (x5)
- net at U?. (in): now also U?. (select); no longer U?. (select)
- net at U?. (in): now also U?.3
- net at U?. (select): now also U?. (in), U?. (select); no longer U?. (in)
- new net: U. (reset), U?. (select) (x3)
- new net: U?. (in), U?. (select) (x15)
- new net: U?. (in), U?. (select), U?. (select) (x2)
- now unconnected: U?. (select), U?. (select), U?. (select), U?. (select), U?. (select)

Commit message: initially integrated processor without being tested
Connections:
- net at U?. (select): now also U?. (in), U?. (select) (x3)
- net at U?. (select): now also U?. (in), U?. (select); no longer U. (reset) (x2)
- net at U?. (select): now also U. (reset); no longer U?. (in) (x5)
- net at U?. (in): now also U?. (select); no longer U?. (select)
- net at U?. (in): now also U?.3
- net at U?. (select): now also U?. (in), U?. (select); no longer U?. (in)
- new net: U. (reset), U?. (select) (x3)
- new net: U?. (in), U?. (select) (x15)
- new net: U?. (in), U?. (select), U?. (select) (x2)
- now unconnected: U?. (select), U?. (select), U?. (select), U?. (select), U?. (select)

Commit message: test12
Connections:
- net at U?. (select): now also U?. (in), U?. (select) (x3)
- net at U?. (select): now also U?. (in), U?. (select); no longer U. (reset) (x2)
- net at U?. (select): now also U. (reset); no longer U?. (in) (x5)
- net at U?. (in): now also U?. (select); no longer U?. (select)
- net at U?. (in): now also U?.3
- net at U?. (select): now also U?. (in), U?. (select); no longer U?. (in)
- new net: U. (reset), U?. (select) (x3)
- new net: U?. (in), U?. (select) (x15)
- new net: U?. (in), U?. (select), U?. (select) (x2)
- now unconnected: U?. (select), U?. (select), U?. (select), U?. (select), U?. (select)
