File: schematics/processorDesign/regFile.kicad_sch (KiCad schematic)
At the start: 31 parts

Commit message: the interrupt is now working correctly
Connections:
- net at U?. (select): now also U?. (in), U?. (select) (x3)
- net at U?. (select): now also U?. (in), U?. (select); no longer U. (reset) (x2)
- net at U?. (select): now also U. (reset); no longer U?. (in) (x5)
- net at U?. (in): now also U?. (select); no longer U?. (select)
- net at U?. (in): now also U?.3
- net at U?. (select): now also U?. (in), U?. (select); no longer U?. (in)
- new net: U. (reset), U?. (select) (x3)
- new net: U?. (in), U?. (select) (x15)
- new net: U?. (in), U?. (select), U?. (select) (x2)
- now unconnected: U?. (select), U?. (select), U?. (select), U?. (select), U?. (select)

Commit message: the processor is now up and running , tested and verified , except for the part related to labels due to a bug in the assembler
Connections:
- net at U?. (select): now also U?. (in), U?. (select) (x3)
- net at U?. (select): now also U?. (in), U?. (select); no longer U. (reset) (x2)
- net at U?. (select): now also U. (reset); no longer U?. (in) (x5)
- net at U?. (in): now also U?. (select); no longer U?. (select)
- net at U?. (in): now also U?.3
- net at U?. (select): now also U?. (in), U?. (select); no longer U?. (in)
- new net: U. (reset), U?. (select) (x3)
- new net: U?. (in), U?. (select) (x15)
- new net: U?. (in), U?. (select), U?. (select) (x2)
- now unconnected: U?. (select), U?. (select), U?. (select), U?. (select), U?. (select)

Commit message: the processor is now up and running , tested and verified completly for almost most of the things
Connections:
- net at U?. (select): now also U?. (in), U?. (select) (x3)
- net at U?. (select): now also U?. (in), U?. (select); no longer U. (reset) (x2)
- net at U?. (select): now also U. (reset); no longer U?. (in) (x5)
- net at U?. (in): now also U?. (select); no longer U?. (select)
- net at U?. (in): now also U?.3
- net at U?. (select): now also U?. (in), U?. (select); no longer U?. (in)
- new net: U. (reset), U?. (select) (x3)
- new net: U?. (in), U?. (select) (x15)
- new net: U?. (in), U?. (select), U?. (select) (x2)
- now unconnected: U?. (select), U?. (select), U?. (select), U?. (select), U?. (select)

Commit message: added small code to EDU
Connections:
- net at U?. (select): now also U?. (in), U?. (select) (x3)
- net at U?. (select): now also U?. (in), U?. (select); no longer U. (reset) (x2)
- net at U?. (select): now also U. (reset); no longer U?. (in) (x5)
- net at U?. (in): now also U?. (select); no longer U?. (select)
- net at U?. (in): now also U?.3
- net at U?. (select): now also U?. (in), U?. (select); no longer U?. (in)
- new net: U. (reset), U?. (select) (x3)
- new net: U?. (in), U?. (select) (x15)
- new net: U?. (in), U?. (select), U?. (select) (x2)
- now unconnected: U?. (select), U?. (select), U?. (select), U?. (select), U?. (select)
