File: schematics/processorDesign/CU.kicad_sch (KiCad schematic)
At the start: 112 parts

Commit message: the interrupt is now working correctly
Parts:
- added U?: equality, symbol computerArchProj:equality
Connections:
- net SET_INT: now also U?.
- net at U?.: now also U?.2 (x4)
- net at U?.: now also U?.1 (x14)
- net at U?. (select): now also U?.2, U?.9
- net at U?.: now also U?.1, U?.1 (x2)
- net at U?. (select): now also U?.3, U?.8
- net at U?. (select): now also U?.3, U?.5
- new net: U?., U?. (select), U?.2
- new net: U?., U?. (select), U?.8
- now unconnected: U?., U?., U?. (select), U?. (select)
Changed lines of the file:
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@@
   (junction (at 722.63 43.18) (diameter 0) (color 0 0 0 0)
   )
+  (junction (at 49.53 708.66) (diameter 0) (color 0 0 0 0)
+  )
   (junction (at 546.1 351.79) (diameter 0) (color 0 0 0 0)
   )
@@
     (stroke (width 0) (type default) (color 255 121 109 1))
   )
-  (wire (pts (xy 207.01 716.28) (xy 207.01 783.59))
-    (stroke (width 0) (type default) (color 90 122 255 1))
+  (wire (pts (xy 204.47 750.57) (xy 204.47 1088.39))
+    (stroke (width 0) (type default) (color 102 130 255 1))
   )
   (wire (pts (xy 736.6 952.5) (xy 737.87 952.5))
@@
     (stroke (width 0) (type default) (color 101 133 255 1))
   )
+  (wire (pts (xy 207.01 716.28) (xy 207.01 783.59))
+    (stroke (width 0) (type default) (color 90 122 255 1))
+  )
   (wire (pts (xy 847.09 118.11) (xy 868.68 118.11))
     (stroke (width 0) (type default) (color 0 0 0 0))
@@
     (stroke (width 0) (type default) (color 0 0 0 0))
   )
+  (wire (pts (xy 843.28 1088.39) (xy 843.28 906.78))
+    (stroke (width 0) (type default) (color 102 130 255 1))
+  )
   (bus (pts (xy 49.53 500.38) (xy 49.53 461.01))
     (stroke (width 0) (type default) (color 0 0 0 0))
@@
     (stroke (width 0) (type default) (color 194 133 255 1))
   )
+  (wire (pts (xy 204.47 1088.39) (xy 843.28 1088.39))
+    (stroke (width 0) (type default) (color 102 130 255 1))
+  )
   (wire (pts (xy 610.87 853.44) (xy 614.68 853.44))
     (stroke (width 0) (type default) (color 71 69 255 1))
@@
     (stroke (width 0) (type default) (color 0 0 0 0))
   )
+  (wire (pts (xy 167.64 750.57) (xy 204.47 750.57))
+    (stroke (width 0) (type default) (color 102 130 255 1))
+  )
   (bus (pts (xy 459.74 257.81) (xy 459.74 193.04))
     (stroke (width 0) (type default) (color 255 106 252 1))
@@
     (stroke (width 0) (type default) (color 0 0 0 0))
   )
+  (wire (pts (xy 843.28 906.78) (xy 1145.54 906.78))
+    (stroke (width 0) (type default) (color 102 130 255 1))
+  )
   (wire (pts (xy 556.26 830.58) (xy 576.58 830.58))
     (stroke (width 0) (type default) (color 0 0 0 0))
@@
     (stroke (width 0) (type default) (color 87 141 108 1))
   )
+  (bus (pts (xy 139.7 758.19) (xy 154.94 758.19))
+    (stroke (width 0) (type default) (color 255 121 109 1))
+  )
   (wire (pts (xy 610.87 850.9) (xy 614.68 850.9))
     (stroke (width 0) (type default) (color 0 0 0 0))
@@
     (stroke (width 0) (type default) (color 180 176 85 1))
   )
+  (bus (pts (xy 154.94 742.95) (xy 49.53 742.95))
+    (stroke (width 0) (type default) (color 0 0 0 0))
+  )
   (wire (pts (xy 612.14 680.72) (xy 612.14 693.42))
     (stroke (width 0) (type default) (color 0 0 0 0))
@@
     (stroke (width 0) (type default) (color 0 0 0 0))
   )
+  (bus (pts (xy 49.53 708.66) (xy 49.53 742.95))
+    (stroke (width 0) (type default) (color 0 0 0 0))
+  )
   (wire (pts (xy 200.66 336.55) (xy 200.66 46.99))
     (stroke (width 0) (type default) (color 184 121 43 1))
@@
     (effects (font (size 1.27 1.27)) (justify left bottom))
   )
+  (text "instr[15:12] 4 bits width (op-code)" (at 118.11 742.95 0)
+    (effects (font (size 1.27 1.27)) (justify left bottom))
+  )
   (text "16 bits width" (at 35.56 457.2 0)
     (effects (font (size 1.27 1.27)) (justify left bottom))
@@
     )
   )
+  (global_label "11 (dec)" (shape input) (at 139.7 758.19 180) (fields_autoplaced)
+    (effects (font (size 1.27 1.27)) (justify right))
+    (property "Intersheet References" "${INTERSHEET_REFS}" (id 0) (at 128.8807 758.1106 0)
+      (effects (font (size 1.27 1.27)) (justify right) hide)
+    )
+  )
   (global_label "1 (dec)" (shape input) (at 528.32 869.95 180) (fields_autoplaced)
     (effects (font (size 1.27 1.27)) (justify right))
@@
     (pin "7")
   )
+  (symbol (lib_id "computerArchProj:equality") (at 162.56 750.57 90) (unit 1)
+    (in_bom yes) (on_board yes)
+    (property "Reference" "U?" (id 0) (at 161.4525 735.33 90)
+      (effects (font (size 1.27 1.27)) hide)
+    )
+    (property "Value" "equality" (id 1) (at 156.21 750.57 0))
+    (property "Footprint" "" (id 2) (at 162.56 750.57 0)
+      (effects (font (size 1.27 1.27)) hide)
+    )
+    (property "Datasheet" "" (id 3) (at 162.56 750.57 0)
+      (effects (font (size 1.27 1.27)) hide)
+    )
+    (pin "")
+    (pin "")
+    (pin "")
+  )
   (symbol (lib_id "computerArchProj:mux_2x1") (at 1070.61 593.09 90) (mirror x) (unit 1)

Commit message: the processor is up and running tested and verified, need only tests for some bonus instructions like all I_types instruction except LDM , MUL , DIV , testing EDU and HDU
Parts:
- added U? (x5): 4071, symbol 4xxx:4071
Connections:
- net PC_push_pop: now also U?.3; no longer U?.3
- net mem_address_src: now also U?.3; no longer U?., U?.1, U?.1, U?.2, U?.2, U?.2, U?.2, U?.2, U?.2
- net mem_data_src: now also U?.3; no longer U?.3
- net at U?.: now also U?.2 (x4)
- net at U?.: now also U?.1 (x14)
- net at U?., U?.2, U?.2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: now also U?.2
- net at U?. (select): now also U?.2, U?.9
- net at U?.: now also U?.1, U?.1 (x2)
- net at U?. (select): now also U?.3, U?.8
- net at U?. (select): now also U?.3, U?.5
- net at U?.1: now also U?.3
- net at U?.3, U?.4: now also U?.1
- new net: U?., U?.1, U?.1, U?.2, U?.2, U?.2, U?.2, U?.2, U?.2, U?.2
- new net: U?.1, U?.1, U?.1, U?.3
- new net: U?.2, U?.3 (x2)
- new net: U?., U?. (select), U?.2
- new net: U?., U?. (select), U?.8
- now unconnected: U?., U?., U?. (select), U?. (select)

Commit message: the processor is now up and running , tested and verified , except for the part related to labels due to a bug in the assembler
Connections:
- net at U?.: now also U?.2 (x4)
- net at U?.: now also U?.1 (x14)
- net at U?. (select): now also U?.2, U?.9
- net at U?.: now also U?.1, U?.1 (x2)
- net at U?. (select): now also U?.3, U?.8
- net at U?. (select): now also U?.3, U?.5
- new net: U?., U?. (select), U?.2
- new net: U?., U?. (select), U?.8
- now unconnected: U?., U?., U?. (select), U?. (select)

Commit message: the processor is now up and running , tested and verified completly for almost most of the things
Parts:
- removed U?: 4075, symbol 4xxx:4075
- added U?: mux_2x1, symbol computerArchProj:mux_2x1
- added U?: mux_4x2, symbol computerArchProj:mux_4x2
- added U?: 4072, symbol 4xxx:4072
- added U? (x2): equality, symbol computerArchProj:equality
Connections:
- net at U?.: now also U?.2 (x4)
- net at U?.: now also U?.1 (x14)
- net at U?. (select): now also U?.2, U?.1
- net at U?.: now also U?.1, U?.1 (x2)
- net at U?. (select): now also U?.3, U?.8
- net at U?.: no longer U?. (select)
- net at U?. (select): no longer U?.
- net at U?. (select): now also U?.3, U?.5
- new net: U?., U?. (select), U?.2
- new net: U?., U?.3
- new net: U?., U?. (select), U?.4
- new net: U?., U?. (select), U?.5
- new net RST: U?.
Other:
- note added: "MOD"

Commit message: added small code to EDU
Connections:
- net at U?.: now also U?.2 (x4)
- net at U?.: now also U?.1 (x14)
- net at U?. (select): now also U?., U?.2
- net at U?. (select): now also U?.1, U?.2
- net at U?.: now also U?.1, U?.1 (x2)
- net at U?. (select): now also U?.3, U?.8
- net at U?. (select): now also U?.3, U?.5
- new net: U?., U?. (select), U?.4
- new net: U?., U?. (select), U?.5
- now unconnected: U?., U?., U?., U?. (select), U?. (select)
